File: kicad/cluster.sch (KiCad schematic (older format))
At the start: 16 parts, among them J1 Conn_01x07

Commit message: Edit cluster board for choc key switch
Parts:
- removed IR3: IR908-7C-F, lalboard:IR908-7C-F, symbol lalboard:IR908-7C-F
- removed PT3: PT908-7B-F, lalboard:PT908-7C-F, symbol lalboard:PT908-7B-F
- removed R3: 270, Resistor_SMD:R_1206_3216Metric_Pad1.42x1.75mm_HandSolder, symbol Device:R
- added SW1: SW_Push, lalboard:SW_CHOC, symbol Switch:SW_Push
- IR1, IR2, IR4, IR5: value IR908-7C-F -> OP140C
- PT1, PT2, PT4, PT5: value PT908-7B-F -> OP550A
- R1, R2, R4, R5: value 270 -> 150
Connections:
- wire segments 0 -> 1
Changed lines of the file:
@@
 EESchema Schematic File Version 4
+LIBS:cluster-cache
 EELAYER 30 0
 EELAYER END
@@
 P 3700 1350
 F 0 "PT1" H 3650 1550 50  0000 L CNN
-F 1 "PT908-7B-F" V 3950 1150 50  0000 L CNN
+F 1 "OP550A" V 3950 1150 50  0000 L CNN
 F 2 "lalboard:PT908-7C-F" H 4180 1210 50  0001 C CNN
 F 3 "https://www.everlight.com/file/ProductFile/PT908-7B-F.pdf" H 3700 1350 50  0001 C CNN
@@
 P 3300 1550
 F 0 "R1" V 3400 1500 50  0000 L CNN
-F 1 "270" V 3294 1474 50  0000 L CNN
+F 1 "150" V 3294 1474 50  0000 L CNN
 F 2 "Resistor_SMD:R_1206_3216Metric_Pad1.42x1.75mm_HandSolder" V 3230 1550 50  0001 C CNN
 F 3 "~" H 3300 1550 50  0001 C CNN
@@
 P 3300 1200
 F 0 "IR1" V 3350 1300 50  0000 C CNN
-F 1 "IR908-7C-F" H 3300 1100 50  0000 C CNN
+F 1 "OP140C" H 3300 1100 50  0000 C CNN
 F 2 "lalboard:IR908-7C-F" H 3300 1375 50  0001 C CNN
 F 3 "https://www.everlight.com/file/ProductFile/201407052136280483.pdf" H 3250 1200 50  0001 C CNN
@@
 P 3700 2650
 F 0 "PT2" H 3650 2850 50  0000 L CNN
-F 1 "PT908-7B-F" V 3950 2450 50  0000 L CNN
+F 1 "OP550A" V 3950 2450 50  0000 L CNN
 F 2 "lalboard:PT908-7C-F" H 4180 2510 50  0001 C CNN
 F 3 "https://www.everlight.com/file/ProductFile/PT908-7B-F.pdf" H 3700 2650 50  0001 C CNN
@@
 P 3300 2850
 F 0 "R2" V 3400 2800 50  0000 L CNN
-F 1 "270" V 3294 2774 50  0000 L CNN
+F 1 "150" V 3294 2774 50  0000 L CNN
 F 2 "Resistor_SMD:R_1206_3216Metric_Pad1.42x1.75mm_HandSolder" V 3230 2850 50  0001 C CNN
 F 3 "~" H 3300 2850 50  0001 C CNN
@@
 P 3300 2500
 F 0 "IR2" V 3350 2600 50  0000 C CNN
-F 1 "IR908-7C-F" H 3300 2400 50  0000 C CNN
+F 1 "OP140C" H 3300 2400 50  0000 C CNN
 F 2 "lalboard:IR908-7C-F" H 3300 2675 50  0001 C CNN
 F 3 "https://www.everlight.com/file/ProductFile/201407052136280483.pdf" H 3250 2500 50  0001 C CNN
@@
 	3050 2100 3050 3300
 $Comp
-L lalboard:PT908-7B-F PT3
-U 1 1 60613592
-P 3700 3950
-F 0 "PT3" H 3650 4150 50  0000 L CNN
-F 1 "PT908-7B-F" V 3950 3750 50  0000 L CNN
-F 2 "lalboard:PT908-7C-F" H 4180 3810 50  0001 C CNN
-F 3 "https://www.everlight.com/file/ProductFile/PT908-7B-F.pdf" H 3700 3950 50  0001 C CNN
-	1    3700 3950
-	1    0    0    -1
-$EndComp
-$Comp
 L power:+5V #PWR0104
 U 1 1 60613598
@@
 	1    0    0    -1
 $EndComp
-Text GLabel 3800 4150 3    50   Input ~ 0
-C3
-$Comp
-L Device:R R3
-U 1 1 6061359F
-P 3300 4150
-F 0 "R3" V 3400 4100 50  0000 L CNN
-F 1 "270" V 3294 4074 50  0000 L CNN
-F 2 "Resistor_SMD:R_1206_3216Metric_Pad1.42x1.75mm_HandSolder" V 3230 4150 50  0001 C CNN
-F 3 "~" H 3300 4150 50  0001 C CNN
-	1    3300 4150
-	-1   0    0    1
-$EndComp
-$Comp
-L lalboard:IR908-7C-F IR3
-U 1 1 606135A5
-P 3300 3800
-F 0 "IR3" V 3350 3900 50  0000 C CNN
-F 1 "IR908-7C-F" H 3300 3700 50  0000 C CNN
-F 2 "lalboard:IR908-7C-F" H 3300 3975 50  0001 C CNN
-F 3 "https://www.everlight.com/file/ProductFile/201407052136280483.pdf" H 3250 3800 50  0001 C CNN
-	1    3300 3800
-	0    1    -1   0
-$EndComp
-$Comp
-L power:GND #PWR0105
-U 1 1 606135AB
-P 3300 4300
-F 0 "#PWR0105" H 3300 4050 50  0001 C CNN
-F 1 "GND" H 3305 4127 50  0000 C CNN
-F 2 "" H 3300 4300 50  0001 C CNN
-F 3 "" H 3300 4300 50  0001 C CNN
-	1    3300 4300
-	1    0    0    -1
-$EndComp
-$Comp
-L power:+5V #PWR0106
-U 1 1 606135B1
-P 3800 3750
-F 0 "#PWR0106" H 3800 3600 50  0001 C CNN
-F 1 "+5V" H 3815 3923 50  0000 C CNN
-F 2 "" H 3800 3750 50  0001 C CNN
-F 3 "" H 3800 3750 50  0001 C CNN
-	1    3800 3750
-	1    0    0    -1
-$EndComp
 Wire Notes Line
 	3050 3400 4100 3400
@@
 P 3700 5250
 F 0 "PT4" H 3650 5450 50  0000 L CNN
-F 1 "PT908-7B-F" V 3950 5050 50  0000 L CNN
+F 1 "OP550A" V 3950 5050 50  0000 L CNN
 F 2 "lalboard:PT908-7C-F" H 4180 5110 50  0001 C CNN
 F 3 "https://www.everlight.com/file/ProductFile/PT908-7B-F.pdf" H 3700 5250 50  0001 C CNN
@@
 P 3300 5450
 F 0 "R4" V 3400 5400 50  0000 L CNN
-F 1 "270" V 3294 5374 50  0000 L CNN
+F 1 "150" V 3294 5374 50  0000 L CNN
 F 2 "Resistor_SMD:R_1206_3216Metric_Pad1.42x1.75mm_HandSolder" V 3230 5450 50  0001 C CNN
 F 3 "~" H 3300 5450 50  0001 C CNN
@@
 P 3300 5100
 F 0 "IR4" V 3350 5200 50  0000 C CNN
-F 1 "IR908-7C-F" H 3300 5000 50  0000 C CNN
+F 1 "OP140C" H 3300 5000 50  0000 C CNN
 F 2 "lalboard:IR908-7C-F" H 3300 5275 50  0001 C CNN
 F 3 "https://www.everlight.com/file/ProductFile/201407052136280483.pdf" H 3250 5100 50  0001 C CNN
@@
 P 3700 6550
 F 0 "PT5" H 3650 6750 50  0000 L CNN
-F 1 "PT908-7B-F" V 3950 6350 50  0000 L CNN
+F 1 "OP550A" V 3950 6350 50  0000 L CNN
 F 2 "lalboard:PT908-7C-F" H 4180 6410 50  0001 C CNN
 F 3 "https://www.everlight.com/file/ProductFile/PT908-7B-F.pdf" H 3700 6550 50  0001 C CNN
@@
 P 3300 6750
 F 0 "R5" V 3400 6700 50  0000 L CNN
-F 1 "270" V 3294 6674 50  0000 L CNN
+F 1 "150" V 3294 6674 50  0000 L CNN
 F 2 "Resistor_SMD:R_1206_3216Metric_Pad1.42x1.75mm_HandSolder" V 3230 6750 50  0001 C CNN
 F 3 "~" H 3300 6750 50  0001 C CNN
@@
 P 3300 6400
 F 0 "IR5" V 3350 6500 50  0000 C CNN
-F 1 "IR908-7C-F" H 3300 6300 50  0000 C CNN
+F 1 "OP140C" H 3300 6300 50  0000 C CNN
 F 2 "lalboard:IR908-7C-F" H 3300 6575 50  0001 C CNN
 F 3 "https://www.everlight.com/file/ProductFile/201407052136280483.pdf" H 3250 6400 50  0001 C CNN
@@
 Text Notes 3850 7150 0    50   ~ 0
 South
+$Comp
+L Switch:SW_Push SW1
+U 1 1 610EC1B0
+P 3300 4000
+F 0 "SW1" V 3254 4148 50  0000 L CNN
+F 1 "SW_Push" V 3345 4148 50  0000 L CNN
+F 2 "lalboard:SW_CHOC" H 3300 4200 50  0001 C CNN
+F 3 "~" H 3300 4200 50  0001 C CNN
+	1    3300 4000
+	0    1    1    0
+$EndComp
+Wire Wire Line
+	3300 3700 3300 3800
+Text GLabel 3300 4200 3    50   Input ~ 0
+C3
 $EndSCHEMATC

Commit message: Customize
Parts:
- added R3: 5.1k, Resistor_SMD:R_0805_2012Metric_Pad1.15x1.40mm_HandSolder, symbol Device:R
Connections:
- wire segments 1 -> 3
Other:
- moved on the sheet: SW1
Changed lines of the file:
@@
 Wire Notes Line
 	3050 2100 3050 3300
-$Comp
-L power:+5V #PWR0104
-U 1 1 60613598
-P 3300 3700
-F 0 "#PWR0104" H 3300 3550 50  0001 C CNN
-F 1 "+5V" H 3315 3873 50  0000 C CNN
-F 2 "" H 3300 3700 50  0001 C CNN
-F 3 "" H 3300 3700 50  0001 C CNN
-	1    3300 3700
-	1    0    0    -1
-$EndComp
 Wire Notes Line
 	3050 3400 4100 3400
@@
 L Switch:SW_Push SW1
 U 1 1 610EC1B0
-P 3300 4000
-F 0 "SW1" V 3254 4148 50  0000 L CNN
-F 1 "SW_Push" V 3345 4148 50  0000 L CNN
-F 2 "lalboard:SW_CHOC" H 3300 4200 50  0001 C CNN
-F 3 "~" H 3300 4200 50  0001 C CNN
-	1    3300 4000
-	0    1    1    0
+P 3700 4100
+F 0 "SW1" V 3654 4248 50  0000 L CNN
+F 1 "SW_Push" V 3745 4248 50  0000 L CNN
+F 2 "lalboard:SW_CHOC" H 3700 4300 50  0001 C CNN
+F 3 "~" H 3700 4300 50  0001 C CNN
+	1    3700 4100
+	1    0    0    -1
 $EndComp
 Wire Wire Line
@@
 Text GLabel 3300 4200 3    50   Input ~ 0
 C3
+$Comp
+L power:GND #PWR05
+U 1 1 6180E9F7
+P 3900 4100
+F 0 "#PWR05" H 3900 3850 50  0001 C CNN
+F 1 "GND" H 3905 3927 50  0000 C CNN
+F 2 "" H 3900 4100 50  0001 C CNN
+F 3 "" H 3900 4100 50  0001 C CNN
+	1    3900 4100
+	1    0    0    -1
+$EndComp
+$Comp
+L power:+5V #PWR04
+U 1 1 6180FA70
+P 3300 3700
+F 0 "#PWR04" H 3300 3550 50  0001 C CNN
+F 1 "+5V" H 3315 3873 50  0000 C CNN
+F 2 "" H 3300 3700 50  0001 C CNN
+F 3 "" H 3300 3700 50  0001 C CNN
+	1    3300 3700
+	1    0    0    -1
+$EndComp
+$Comp
+L Device:R R3
+U 1 1 618104DA
+P 3300 3950
+F 0 "R3" V 3400 3900 50  0000 L CNN
+F 1 "5.1k" V 3294 3874 50  0000 L CNN
+F 2 "Resistor_SMD:R_0805_2012Metric_Pad1.15x1.40mm_HandSolder" V 3230 3950 50  0001 C CNN
+F 3 "~" H 3300 3950 50  0001 C CNN
+	1    3300 3950
+	-1   0    0    1
+$EndComp
+Wire Wire Line
+	3500 4100 3300 4100
+Wire Wire Line
+	3300 4100 3300 4200
+Connection ~ 3300 4100
+$Comp
+L power:PWR_FLAG #FLG0101
+U 1 1 618111FE
+P 2000 3600
+F 0 "#FLG0101" H 2000 3675 50  0001 C CNN
+F 1 "PWR_FLAG" H 2000 3773 50  0000 C CNN
+F 2 "" H 2000 3600 50  0001 C CNN
+F 3 "~" H 2000 3600 50  0001 C CNN
+	1    2000 3600
+	-1   0    0    1
+$EndComp
+Connection ~ 2000 3600
+$Comp
+L power:PWR_FLAG #FLG0102
+U 1 1 61812256
+P 2000 3000
+F 0 "#FLG0102" H 2000 3075 50  0001 C CNN
+F 1 "PWR_FLAG" H 2000 3173 50  0000 C CNN
+F 2 "" H 2000 3000 50  0001 C CNN
+F 3 "~" H 2000 3000 50  0001 C CNN
+	1    2000 3000
+	1    0    0    -1
+$EndComp
+Connection ~ 2000 3000
 $EndSCHEMATC
