File: kicad/main_board.sch (KiCad schematic (older format))
At the start: 56 parts, among them J1 Conn_01x07, J2 Conn_01x07, J3 Conn_01x07, J4 Conn_01x07, J5 Conn_01x07, J6 TYPE-C-31-M-12, J7 TYPE-C-31-M-12, J8 Conn_01x07, Q1 Q_NPN_BEC, Q2 Q_NPN_BEC, Q3 Q_NPN_BEC, Q4 Q_NPN_BEC, Q5 Q_NPN_BEC, SW1 Reset, SW2 Boot, U1 esp32-s2-wroom, U2 XC6220B331MR, U3 USBLC6-2SC6, U4 USBLC6-2SC6, U5 LMV324, U6 LMV324

Commit message: wip: update mainboard with STM32
Parts:
- removed C1: 10u, Capacitor_SMD:C_0805_2012Metric_Pad1.15x1.40mm_HandSolder, symbol Device:C_Small
- removed C2, C5: .1u, Capacitor_SMD:C_0805_2012Metric_Pad1.15x1.40mm_HandSolder, symbol Device:C_Small
- removed C3: 1u, Capacitor_SMD:C_0805_2012Metric_Pad1.15x1.40mm_HandSolder, symbol Device:C_Small
- removed FB4: ACML-0805-500-T, Inductor_SMD:L_0805_2012Metric_Pad1.15x1.40mm_HandSolder, symbol Device:Ferrite_Bead_Small
- removed R1, R2: 10k, Resistor_SMD:R_0805_2012Metric_Pad1.15x1.40mm_HandSolder, symbol Device:R_Small
- removed R19, R20: 22, Resistor_SMD:R_0805_2012Metric_Pad1.15x1.40mm_HandSolder, symbol Device:R_Small
- removed U1: esp32-s2-wroom, lalboard:ESP32-S2-WROOM-handsoldering, symbol lalboard:esp32-s2-wroom
- removed U2: XC6220B331MR, Package_TO_SOT_SMD:SOT-23-5, symbol Regulator_Linear:XC6220B331MR
- added C1, C10, C2, C3, C5: 0.1u, Capacitor_SMD:C_0805_2012Metric_Pad1.18x1.45mm_HandSolder, symbol Device:C
- added F1: Polyfuse 100mA, Fuse:Fuse_1210_3225Metric_Pad1.42x2.65mm_HandSolder, symbol Device:Polyfuse
- added H3: SWDIO, MountingHole:MountingHole_2.2mm_M2_Pad, symbol Mechanical:MountingHole_Pad
- added H4: SWCLK, MountingHole:MountingHole_2.2mm_M2_Pad, symbol Mechanical:MountingHole_Pad
- added R1: 10k, Resistor_SMD:R_0805_2012Metric_Pad1.20x1.40mm_HandSolder, symbol Device:R
- added U1: MIC5504-3.3YM5, Package_TO_SOT_SMD:SOT-23-5, symbol Regulator_Linear:MIC5504-3.3YM5
- added U2: STM32L412C8T6, Package_QFP:TQFP-48_7x7mm_P0.5mm, symbol lalboard:STM32L412C8T6
- C4, C8, C9: footprint Capacitor_SMD:C_0805_2012Metric_Pad1.15x1.40mm_HandSolder -> Capacitor_SMD:C_0805_2012Metric_Pad1.18x1.45mm_HandSolder
- C6: value 10u -> 1uF; footprint Capacitor_SMD:C_0805_2012Metric_Pad1.15x1.40mm_HandSolder -> Capacitor_SMD:C_0805_2012Metric_Pad1.18x1.45mm_HandSolder
- C7: value 4.7u -> 1uF; footprint Capacitor_SMD:C_0805_2012Metric_Pad1.15x1.40mm_HandSolder -> Capacitor_SMD:C_0805_2012Metric_Pad1.18x1.45mm_HandSolder
- J6, J7: symbol Connector:USB_C_Receptacle_USB2.0 -> main_board-rescue:USB_C_Receptacle_USB2.0-Connector
Connections:
- net labels added: BOOT0, I2C_SCL, I2C_SDA, NRST, SCL_raw, SDA_raw, SWCLK, SWDIO, USB_D+, USB_D-, VBUS
- net labels removed: CHIP_PU, D+, D-, GPIO_0, U1RX, U1RX_raw, U1TX, U1TX_raw
- wire segments 137 -> 149
- no-connect marks 4 -> 25
Other:
- moved on the sheet: SW2

Commit message: Update kicad pcb data to change parts
Parts:
- added H5, H6: MountingHole_Pad, TestPoint:TestPoint_THTPad_D2.0mm_Drill1.0mm, symbol Mechanical:MountingHole_Pad
- added R19, R2: 5.1k, Resistor_SMD:R_0805_2012Metric_Pad1.15x1.40mm_HandSolder, symbol Device:R
- C1, C10, C2, C3, C4, C5, C6, C7, C8, C9: footprint Capacitor_SMD:C_0805_2012Metric_Pad1.18x1.45mm_HandSolder -> Capacitor_SMD:C_0805_2012Metric_Pad1.15x1.40mm_HandSolder
- H3, H4: footprint MountingHole:MountingHole_2.2mm_M2_Pad -> TestPoint:TestPoint_THTPad_D2.0mm_Drill1.0mm
- J6: value TYPE-C-31-M-12 -> USB-C; footprint Connector_USB:USB_C_Receptacle_HRO_TYPE-C-31-M-12 -> lalboard:GCT_USB4110-GF-A_REVB; symbol main_board-rescue:USB_C_Receptacle_USB2.0-Connector -> lalboard:USB4110-GF-A_REVB
- J7: footprint Connector_USB:USB_C_Receptacle_HRO_TYPE-C-31-M-12 -> lalboard:GCT_USB4110-GF-A_REVB; symbol main_board-rescue:USB_C_Receptacle_USB2.0-Connector -> lalboard:USB4110-GF-A_REVB
- R1: value 10k -> 5.1k; footprint Resistor_SMD:R_0805_2012Metric_Pad1.20x1.40mm_HandSolder -> Resistor_SMD:R_0805_2012Metric_Pad1.15x1.40mm_HandSolder
- SW1, SW2: footprint Button_Switch_THT:SW_PUSH_6mm_H5mm -> Button_Switch_SMD:SW_SPST_B3U-1000P
- U3, U4: symbol Power_Protection:USBLC6-2SC6 -> main_board-rescue:USBLC6-2SC6-Power_Protection
Connections:
- net +3V3: now also H5.1, R19.1, R2.1
- net BOOT0: now also H6.1
- net GND: now also R17.1, R18.1; no longer J6.A1 (GND), J6.A12 (GND), J6.B1 (GND), J6.B12 (GND), J7.A1 (GND), J7.A12 (GND), J7.B1 (GND), J7.B12 (GND), R17.2, R18.2
- net I2C_SCL: now also R2.2
- net I2C_SDA: now also R19.2
- net VBUS: now also J6.A4/B9 (VBUS), J6.B4/A9 (VBUS), J7.A4/B9 (VBUS), J7.B4/A9 (VBUS); no longer J6.A4 (VBUS), J6.A9 (VBUS), J6.B4 (VBUS), J6.B9 (VBUS), J7.A4 (VBUS), J7.A9 (VBUS), J7.B4 (VBUS), J7.B9 (VBUS)
- net at FB1.1, J6.S1 (GND): now also J6.A1/B12 (GND), J6.B1/A12 (GND), J6.S2 (GND), J6.S3 (GND), J6.S4 (GND)
- net at J7.A5 (CC1): now also R17.2; no longer R18.1
- net at J7.B5 (CC2): now also R18.2; no longer R17.1
- net at FB3.1, J7.S1 (GND): now also J7.A1/B12 (GND), J7.B1/A12 (GND), J7.S2 (GND), J7.S3 (GND), J7.S4 (GND)
Other:
- moved on the sheet: FB3, R15, R16, R17, R18

Commit message: Customize
Parts:
- removed Q1, Q2, Q3, Q4, Q5: Q_NPN_BEC, Package_TO_SOT_SMD:SOT-23_Handsoldering, symbol Device:Q_NPN_BEC
- added JP1: SolderJumper_2_Open, Jumper:SolderJumper-2_P1.3mm_Open_RoundedPad1.0x1.5mm, symbol Jumper:SolderJumper_2_Open
- added Q1, Q2, Q3: Q_DUAL_NMOS_S1G1D2S2G2D1, Package_TO_SOT_SMD:SOT-363_SC-70-6_Handsoldering, symbol Device:Q_DUAL_NMOS_S1G1D2S2G2D1
- added unit 1 of U6
- added unit 3 of U6
- added unit 4 of U6
- R10, R11, R12, R13, R14: value 1.5k -> 5.1k
Connections:
- net AMP_REF: now also U6.10 (+), U6.12 (+), U6.3 (+)
- net COL3: now also R9.2, U6.6 (-), JP1.1 (A); no longer R7.2, U5.9 (-)
- net COL3_AMP: now also R9.1, U2.41 (PB5), U6.7, JP1.2 (B); no longer R7.1, U2.39 (PB3), U5.8
- net COL5: now also R7.2, U5.9 (-); no longer R9.2, U6.6 (-)
- net COL5_AMP: now also R7.1, U2.39 (PB3), U5.8; no longer R9.1, U2.41 (PB5), U6.7
- net GND: now also R10.2, R11.2, R12.2, R13.2, R14.2, Q1.1 (S), Q1.4 (S), Q2.1 (S), Q2.4 (S), Q3.1 (S), Q3.3 (D), Q3.4 (S), Q3.5 (G)
- net ROW1: now also R14.1, Q3.2 (G); no longer R14.2
- net ROW2: now also R13.1, Q2.5 (G); no longer R13.2
- net ROW3: now also R12.1, Q2.2 (G); no longer R12.2
- net ROW4: now also R11.1, Q1.5 (G); no longer R11.2
- net ROW5: now also R10.1, Q1.2 (G); no longer R10.2
- net at J1.1 (Pin_1): now also Q1.6 (D)
- net at J2.1 (Pin_1): now also Q1.3 (D)
- net at J3.1 (Pin_1): now also Q2.6 (D)
- net at J4.1 (Pin_1): now also Q2.3 (D)
- net at J5.1 (Pin_1): now also Q3.6 (D)
- new net: U6.1, U6.2 (-)
- new net: U6.8, U6.9 (-)
- new net: U6.13 (-), U6.14
Other:
- moved on the sheet: C1, C10, C2, C3, C4, C5, C6, C7, C8, C9, F1, FB1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
