File: kicad/thumb_cluster_right.sch (KiCad schematic (older format))
At the start: 18 parts, among them J1 Conn_01x07

Commit message: Customize
Parts:
- removed IR3: IR908-7C-F, lalboard:IR908-7C-F, symbol lalboard:IR908-7C-F
- removed PT3: PT908-7B-F, lalboard:PT908-7C-F, symbol lalboard:PT908-7B-F
- added SW1: SW_Push-Switch, symbol main_board-rescue:SW_Push-Switch
- added SW2: SW_Push, symbol Switch:SW_Push
- R3: value 120 -> 5.1k; footprint Resistor_SMD:R_1206_3216Metric_Pad1.42x1.75mm_HandSolder -> (none)
Connections:
- wire segments 0 -> 4
Changed lines of the file:
@@
 Wire Notes Line
 	3050 2100 3050 3300
-$Comp
-L lalboard:PT908-7B-F PT3
-U 1 1 60613592
-P 3700 3950
-F 0 "PT3" H 3650 4150 50  0000 L CNN
-F 1 "PT908-7B-F" V 3950 3750 50  0000 L CNN
-F 2 "lalboard:PT908-7C-F" H 4180 3810 50  0001 C CNN
-F 3 "https://www.everlight.com/file/ProductFile/PT908-7B-F.pdf" H 3700 3950 50  0001 C CNN
-	1    3700 3950
-	1    0    0    -1
-$EndComp
-$Comp
-L power:+5V #PWR0104
-U 1 1 60613598
-P 3300 3700
-F 0 "#PWR0104" H 3300 3550 50  0001 C CNN
-F 1 "+5V" H 3315 3873 50  0000 C CNN
-F 2 "" H 3300 3700 50  0001 C CNN
-F 3 "" H 3300 3700 50  0001 C CNN
-	1    3300 3700
-	1    0    0    -1
-$EndComp
-Text GLabel 3800 4150 3    50   Input ~ 0
+Text GLabel 3250 4150 3    50   Input ~ 0
 C3
-$Comp
-L Device:R R3
-U 1 1 6061359F
-P 3300 4150
-F 0 "R3" V 3400 4100 50  0000 L CNN
-F 1 "120" V 3294 4074 50  0000 L CNN
-F 2 "Resistor_SMD:R_1206_3216Metric_Pad1.42x1.75mm_HandSolder" V 3230 4150 50  0001 C CNN
-F 3 "~" H 3300 4150 50  0001 C CNN
-	1    3300 4150
-	-1   0    0    1
-$EndComp
-$Comp
-L lalboard:IR908-7C-F IR3
-U 1 1 606135A5
-P 3300 3800
-F 0 "IR3" V 3350 3900 50  0000 C CNN
-F 1 "IR908-7C-F" H 3300 3700 50  0000 C CNN
-F 2 "lalboard:IR908-7C-F" H 3300 3975 50  0001 C CNN
-F 3 "https://www.everlight.com/file/ProductFile/201407052136280483.pdf" H 3250 3800 50  0001 C CNN
-	1    3300 3800
-	0    1    -1   0
-$EndComp
-$Comp
-L power:GND #PWR0105
-U 1 1 606135AB
-P 3300 4300
-F 0 "#PWR0105" H 3300 4050 50  0001 C CNN
-F 1 "GND" H 3305 4127 50  0000 C CNN
-F 2 "" H 3300 4300 50  0001 C CNN
-F 3 "" H 3300 4300 50  0001 C CNN
-	1    3300 4300
-	1    0    0    -1
-$EndComp
-$Comp
-L power:+5V #PWR0106
-U 1 1 606135B1
-P 3800 3750
-F 0 "#PWR0106" H 3800 3600 50  0001 C CNN
-F 1 "+5V" H 3815 3923 50  0000 C CNN
-F 2 "" H 3800 3750 50  0001 C CNN
-F 3 "" H 3800 3750 50  0001 C CNN
-	1    3800 3750
-	1    0    0    -1
-$EndComp
 Wire Notes Line
 	3050 3400 4100 3400
@@
 Text Notes 3850 7150 0    50   ~ 0
 Mode
+$Comp
+L power:+5V #PWR0104
+U 1 1 61A3D902
+P 3250 3850
+F 0 "#PWR0104" H 3250 3700 50  0001 C CNN
+F 1 "+5V" H 3265 4023 50  0000 C CNN
+F 2 "" H 3250 3850 50  0001 C CNN
+F 3 "" H 3250 3850 50  0001 C CNN
+	1    3250 3850
+	1    0    0    -1
+$EndComp
+$Comp
+L Device:R R3
+U 1 1 61A3E018
+P 3250 4000
+F 0 "R3" H 3320 4046 50  0000 L CNN
+F 1 "5.1k" H 3320 3955 50  0000 L CNN
+F 2 "" V 3180 4000 50  0001 C CNN
+F 3 "~" H 3250 4000 50  0001 C CNN
+	1    3250 4000
+	1    0    0    -1
+$EndComp
+$Comp
+L main_board-rescue:SW_Push-Switch SW1
+U 1 1 61A3F28A
+P 3700 3900
+F 0 "SW1" H 3700 4185 50  0000 C CNN
+F 1 "SW_Push-Switch" H 3700 4094 50  0000 C CNN
+F 2 "" H 3700 4100 50  0001 C CNN
+F 3 "" H 3700 4100 50  0001 C CNN
+	1    3700 3900
+	1    0    0    -1
+$EndComp
+$Comp
+L Switch:SW_Push SW2
+U 1 1 61A40010
+P 3700 4100
+F 0 "SW2" H 3700 4385 50  0000 C CNN
+F 1 "SW_Push" H 3700 4294 50  0000 C CNN
+F 2 "" H 3700 4300 50  0001 C CNN
+F 3 "~" H 3700 4300 50  0001 C CNN
+	1    3700 4100
+	1    0    0    -1
+$EndComp
+Wire Wire Line
+	3250 4150 3500 4150
+Wire Wire Line
+	3500 4150 3500 4100
+Wire Wire Line
+	3500 3900 3500 4100
+Connection ~ 3500 4100
+Wire Wire Line
+	3900 3900 3900 4100
+$Comp
+L power:GND #PWR0105
+U 1 1 61A41A21
+P 3900 4100
+F 0 "#PWR0105" H 3900 3850 50  0001 C CNN
+F 1 "GND" H 3905 3927 50  0000 C CNN
+F 2 "" H 3900 4100 50  0001 C CNN
+F 3 "" H 3900 4100 50  0001 C CNN
+	1    3900 4100
+	1    0    0    -1
+$EndComp
+Connection ~ 3900 4100
 $EndSCHEMATC
